File: Akashi-01.kicad_pcb (KiCad board)
At the start: 2 copper layers, 71.1 x 67.3 mm, 33 parts, among them CN10 PPPC192LFBN-RC, CN7 PPPC192LFBN-RC, SW1 PEC11R-4220F-S0024

Commit message: Silk updated.
Issue 11 : The Silk have to be updated
https://github.com/suikan4github/Akashi-01/issues/11
Other:
- board text added: "Akashi-01 v1.0.4 A Murasaki JIG for Nucleo 64 (C) Seiichi Horie 2019 https://github.com/suikan4github/Akashi-01"
- board text removed: "Akashi-01 v1.0.2 A Murasaki JIG for Nucleo 64 (C) Seiichi Horie 2019 https://github.com/suikan4github/Akashi-01"
Changed lines of the file:
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@@
     (effects (font (size 1 1) (thickness 0.15)))
   )
-  (gr_text "Akashi-01 v1.0.2\nA Murasaki JIG for Nucleo 64\n(C) Seiichi Horie 2019\nhttps://github.com/suikan4github/Akashi-01" (at 175.895 60.96) (layer B.SilkS)
+  (gr_text "Akashi-01 v1.0.4\nA Murasaki JIG for Nucleo 64\n(C) Seiichi Horie 2019\nhttps://github.com/suikan4github/Akashi-01" (at 175.895 60.96) (layer B.SilkS)
     (effects (font (size 1.5 1.5) (thickness 0.15)) (justify left mirror))
   )
